File: potmux.kicad_pcb (KiCad board)
At the start: 2 copper layers, 22.9 x 26.7 mm, 8 parts, among them P1 SOCKET_LEFT, P2 KEYMAN64, P3 SOCKET_RIGHT, U1 4052, U2 4052

Commit message: Licensed under CERN OHL v.1.2
Other:
- board text added: "Licensed under CERN OHL v.1.2 www.henning-bekel.de/potmux"
- board text removed: "Licensed under CERN OSH v.1.2"
Changed lines of the file:
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@@
-(kicad_pcb (version 4) (host pcbnew 4.0.4-stable)
+(kicad_pcb (version 4) (host pcbnew 4.0.3-stable)
   (general
     (links 35)
     (no_connects 1)
-    (area 130.734999 87.554999 153.745001 114.375001)
+    (area 126.165238 80.564999 174.219999 132.240001)
     (thickness 1.6)
     (drawings 26)
@@
     (date 2016-10-24)
     (rev 1)
-    (company "Henning Bekel")
-    (comment 1 "Licensed under CERN OHL v.1.2")
+    (comment 2 "Copyright Henning Bekel 2016.\\nThis documentation describes Open Hardware and is licensed under the CERN OHL v. 1.2.\\nYou may redistribute and modify this documentation under the terms of the CERN OHL v.1.2.\\n(http://ohwr.org/cernohl). This documentation is distributed WITHOUT ANY EXPRESS OR\\nIMPLIED WARRANTY, INCLUDING OF MERCHANTABILITY, SATISFACTORY QUALITY AND FITNESS\\nFOR A PARTICULAR PURPOSE. Please see the CERN OHL v.1.2 for applicable conditions")
   )
   (layers
@@
     )
   )
-  (gr_text "Licensed under CERN OSH v.1.2" (at 137.16 102.87 90) (layer F.SilkS)
+  (gr_text "Licensed under CERN OHL v.1.2\nwww.henning-bekel.de/potmux" (at 137.16 102.87 90) (layer F.SilkS)
     (effects (font (size 0.6 0.6) (thickness 0.15)))
   )
-  (gr_text "PotMux Rev.1 \n©2016 Henning Bekel" (at 135.255 102.87 90) (layer F.SilkS)
+  (gr_text "PotMux Rev.1 \n©2016 Henning Bekel" (at 134.62 102.87 90) (layer F.SilkS)
     (effects (font (size 0.75 0.75) (thickness 0.15)))
   )
@@
   (segment (start 146.6613 97.7089) (end 149.2824 100.33) (width 0.25) (layer B.Cu) (net 3))
   (segment (start 144.2212 97.7089) (end 146.6613 97.7089) (width 0.25) (layer B.Cu) (net 3))
-  (segment (start 152.4 106.68) (end 151.8412 106.68) (width 0.25) (layer B.Cu) (net 4) (status C00000))
-  (segment (start 151.8412 106.68) (end 150.6461 105.4849) (width 0.25) (layer B.Cu) (net 4) (status 400000))
+  (segment (start 152.4 106.68) (end 151.8412 106.68) (width 0.25) (layer B.Cu) (net 4))
+  (segment (start 151.8412 106.68) (end 150.6461 105.4849) (width 0.25) (layer B.Cu) (net 4))
   (segment (start 144.6784 100.2489) (end 143.4289 100.2489) (width 0.25) (layer B.Cu) (net 4))
   (segment (start 143.4289 100.2489) (end 142.24 99.06) (width 0.25) (layer B.Cu) (net 4))
@@
   (segment (start 150.5016 105.4849) (end 150.0632 105.4849) (width 0.25) (layer B.Cu) (net 4))
   (segment (start 150.0632 105.4849) (end 142.9512 105.4849) (width 0.25) (layer B.Cu) (net 4))
-  (segment (start 137.8934 105.3116) (end 135.7916 105.3116) (width 0.25) (layer B.Cu) (net 5))
-  (segment (start 135.7916 105.3116) (end 132.08 101.6) (width 0.25) (layer B.Cu) (net 5) (status 800000))
+  (segment (start 138.303 105.3084) (end 135.7916 105.3116) (width 0.25) (layer B.Cu) (net 5))
+  (segment (start 135.7916 105.3116) (end 132.08 101.6) (width 0.25) (layer B.Cu) (net 5))
   (segment (start 142.24 101.6) (end 142.24 102.235) (width 0.25) (layer F.Cu) (net 5))
   (segment (start 142.24 102.235) (end 140.8489 103.6261) (width 0.25) (layer F.Cu) (net 5))
-  (via (at 137.8934 105.3116) (size 0.6) (layers F.Cu B.Cu) (net 5))
+  (via (at 138.303 105.3084) (size 0.6) (layers F.Cu B.Cu) (net 5))
   (segment (start 144.78 101.6) (end 142.24 101.6) (width 0.25) (layer B.Cu) (net 5))
-  (segment (start 140.1603 105.3116) (end 137.8934 105.3116) (width 0.25) (layer F.Cu) (net 5))
+  (segment (start 140.1603 105.3116) (end 138.303 105.3084) (width 0.25) (layer F.Cu) (net 5))
   (segment (start 140.8489 104.623) (end 140.1603 105.3116) (width 0.25) (layer F.Cu) (net 5))
   (segment (start 140.8489 103.6261) (end 140.8489 104.623) (width 0.25) (layer F.Cu) (net 5))
@@
   (segment (start 149.86 107.95) (end 147.066 107.95) (width 0.25) (layer B.Cu) (net 13))
   (segment (start 151.13 107.95) (end 152.4 109.22) (width 0.25) (layer B.Cu) (net 13))
-  (segment (start 132.08 99.06) (end 137.9474 99.06) (width 0.25) (layer B.Cu) (net 14) (status 400000))
+  (segment (start 132.08 99.06) (end 137.9474 99.06) (width 0.25) (layer B.Cu) (net 14))
   (segment (start 137.9474 99.06) (end 139.0727 100.1853) (width 0.25) (layer B.Cu) (net 14))
   (segment (start 146.725 104.14) (end 149.86 104.14) (width 0.25) (layer B.Cu) (net 14))
@@
   (segment (start 139.0727 100.1853) (end 139.9022 100.1853) (width 0.25) (layer B.Cu) (net 14))
   (segment (start 138.5577 107.1626) (end 138.5577 105.9427) (width 0.25) (layer B.Cu) (net 15))
-  (segment (start 140.8684 102.7684) (end 139.7 101.6) (width 0.25) (layer B.Cu) (net 15) (status 800000))
+  (segment (start 140.8684 102.7684) (end 139.7 101.6) (width 0.25) (layer B.Cu) (net 15))
   (segment (start 140.8684 104.875202) (end 140.8684 102.7684) (width 0.25) (layer B.Cu) (net 15))
   (segment (start 140.359002 105.3846) (end 140.8684 104.875202) (width 0.25) (layer B.Cu) (net 15))
