File: potmux.sch (KiCad schematic (older format))
At the start: 8 parts, among them P1 SOCKET_LEFT, P2 KEYMAN64, P3 SOCKET_RIGHT, U1 4052, U2 4052

Commit message: Revision 2, updated gerber files for production
This revision moves the pin header to the bottom.
Parts:
- removed P2: KEYMAN64, Pin_Headers:Pin_Header_Angled_1x06, symbol CONN_01X06
- added P4: KEYMAN64, Pin_Headers:Pin_Header_Angled_1x06_Pitch2.54mm, symbol CONN_01X06
- C1, C2: footprint Capacitors_ThroughHole:C_Disc_D3_P2.5 -> Capacitors_ThroughHole:C_Disc_D3.0mm_W1.6mm_P2.50mm
- U1, U2: footprint Housings_DIP:DIP-16_W7.62mm -> custom:DIP-16_W7.62mm
Connections:
- net A1: now also P4.6 (P6)
- net A2: now also P4.5 (P5)
- net B1: now also P4.4 (P4)
- net B2: now also P4.3 (P3)
- net GND: now also P4.1 (P1)
- net ~EN: now also P4.2 (P2)
Changed lines of the file:
@@
 Sheet 1 1
 Title "PotMux - Pot line multiplexer for the C64"
-Date "2016-10-24"
-Rev "1"
+Date "2017-04-27"
+Rev "2"
 Comp ""
 Comment1 ""
@@
 POTAX
 $Comp
-L CONN_01X06 P2
-U 1 1 580E7C4B
-P 1550 3050
-F 0 "P2" H 1550 3400 50  0000 C CNN
-F 1 "KEYMAN64" V 1650 3050 50  0000 C CNN
-F 2 "Pin_Headers:Pin_Header_Angled_1x06" H 1550 3050 50  0001 C CNN
-F 3 "" H 1550 3050 50  0000 C CNN
-	1    1550 3050
-	1    0    0    -1
-$EndComp
-Text Label 1350 2800 2    60   ~ 0
-A1
-Text Label 1350 2900 2    60   ~ 0
-A2
-Text Label 1350 3000 2    60   ~ 0
-B1
-Text Label 1350 3100 2    60   ~ 0
-B2
-Text Label 1350 3200 2    60   ~ 0
-~EN
-$Comp
-L GND #PWR02
-U 1 1 580E7E79
-P 1350 3300
-F 0 "#PWR02" H 1350 3050 50  0001 C CNN
-F 1 "GND" H 1350 3150 50  0000 C CNN
-F 2 "" H 1350 3300 50  0000 C CNN
-F 3 "" H 1350 3300 50  0000 C CNN
-	1    1350 3300
-	1    0    0    -1
-$EndComp
-$Comp
-L PWR_FLAG #FLG03
+L PWR_FLAG #FLG02
 U 1 1 580E7FAD
 P 750 7500
-F 0 "#FLG03" H 750 7595 50  0001 C CNN
+F 0 "#FLG02" H 750 7595 50  0001 C CNN
 F 1 "PWR_FLAG" H 750 7680 50  0000 C CNN
 F 2 "" H 750 7500 50  0000 C CNN
@@
 $EndComp
 $Comp
-L PWR_FLAG #FLG04
+L PWR_FLAG #FLG03
 U 1 1 580E7FCA
 P 1200 7500
-F 0 "#FLG04" H 1200 7595 50  0001 C CNN
+F 0 "#FLG03" H 1200 7595 50  0001 C CNN
 F 1 "PWR_FLAG" H 1200 7680 50  0000 C CNN
 F 2 "" H 1200 7500 50  0000 C CNN
@@
 $EndComp
 $Comp
-L GND #PWR05
+L GND #PWR04
 U 1 1 580E8032
 P 1200 7500
-F 0 "#PWR05" H 1200 7250 50  0001 C CNN
+F 0 "#PWR04" H 1200 7250 50  0001 C CNN
 F 1 "GND" H 1200 7350 50  0000 C CNN
 F 2 "" H 1200 7500 50  0000 C CNN
@@
 $EndComp
 $Comp
-L VCC #PWR06
+L VCC #PWR05
 U 1 1 580E8048
 P 750 7500
-F 0 "#PWR06" H 750 7350 50  0001 C CNN
+F 0 "#PWR05" H 750 7350 50  0001 C CNN
 F 1 "VCC" H 750 7650 50  0000 C CNN
 F 2 "" H 750 7500 50  0000 C CNN
@@
 F 0 "U1" H 4600 1950 50  0000 C CNN
 F 1 "4052" H 4600 1750 50  0000 C CNN
-F 2 "Housings_DIP:DIP-16_W7.62mm" H 4500 1950 60  0001 C CNN
+F 2 "custom:DIP-16_W7.62mm" H 4500 1950 60  0001 C CNN
 F 3 "" H 4500 1950 60  0001 C CNN
 	1    4500 1950
@@
 POTAY
 $Comp
-L GND #PWR07
+L GND #PWR06
 U 1 1 580E82C2
 P 5200 2450
-F 0 "#PWR07" H 5200 2200 50  0001 C CNN
+F 0 "#PWR06" H 5200 2200 50  0001 C CNN
 F 1 "GND" H 5200 2300 50  0000 C CNN
 F 2 "" H 5200 2450 50  0000 C CNN
@@
 $EndComp
 $Comp
-L GND #PWR08
+L GND #PWR07
 U 1 1 580E82E0
 P 3800 2250
-F 0 "#PWR08" H 3800 2000 50  0001 C CNN
+F 0 "#PWR07" H 3800 2000 50  0001 C CNN
 F 1 "GND" H 3800 2100 50  0000 C CNN
 F 2 "" H 3800 2250 50  0000 C CNN
@@
 F 0 "U2" H 4600 3800 50  0000 C CNN
 F 1 "4052" H 4600 3600 50  0000 C CNN
-F 2 "Housings_DIP:DIP-16_W7.62mm" H 4500 3800 60  0001 C CNN
+F 2 "custom:DIP-16_W7.62mm" H 4500 3800 60  0001 C CNN
 F 3 "" H 4500 3800 60  0001 C CNN
 	1    4500 3800
@@
 POTBY
 $Comp
-L GND #PWR09
+L GND #PWR08
 U 1 1 580E84A4
 P 5200 4300
-F 0 "#PWR09" H 5200 4050 50  0001 C CNN
+F 0 "#PWR08" H 5200 4050 50  0001 C CNN
 F 1 "GND" H 5200 4150 50  0000 C CNN
 F 2 "" H 5200 4300 50  0000 C CNN
@@
 $EndComp
 $Comp
-L GND #PWR010
+L GND #PWR09
 U 1 1 580E84FF
 P 3800 4100
-F 0 "#PWR010" H 3800 3850 50  0001 C CNN
+F 0 "#PWR09" H 3800 3850 50  0001 C CNN
 F 1 "GND" H 3800 3950 50  0000 C CNN
 F 2 "" H 3800 4100 50  0000 C CNN
@@
 Connection ~ 3350 4300
 $Comp
-L VCC #PWR011
+L VCC #PWR010
 U 1 1 580E897D
 P 3350 4000
-F 0 "#PWR011" H 3350 3850 50  0001 C CNN
+F 0 "#PWR010" H 3350 3850 50  0001 C CNN
 F 1 "VCC" H 3350 4150 50  0000 C CNN
 F 2 "" H 3350 4000 50  0000 C CNN
@@
 $EndComp
 $Comp
-L VCC #PWR012
+L VCC #PWR011
 U 1 1 580E8B82
 P 6200 1850
-F 0 "#PWR012" H 6200 1700 50  0001 C CNN
+F 0 "#PWR011" H 6200 1700 50  0001 C CNN
 F 1 "VCC" H 6200 2000 50  0000 C CNN
 F 2 "" H 6200 1850 50  0000 C CNN
@@
 F 0 "C1" H 6210 2020 50  0000 L CNN
 F 1 "100n" H 6210 1870 50  0000 L CNN
-F 2 "Capacitors_ThroughHole:C_Disc_D3_P2.5" H 6200 1950 50  0001 C CNN
+F 2 "Capacitors_ThroughHole:C_Disc_D3.0mm_W1.6mm_P2.50mm" H 6200 1950 50  0001 C CNN
 F 3 "" H 6200 1950 50  0000 C CNN
 	1    6200 1950
@@
 $EndComp
 $Comp
-L GND #PWR013
+L GND #PWR012
 U 1 1 580E8C87
 P 6200 2050
-F 0 "#PWR013" H 6200 1800 50  0001 C CNN
+F 0 "#PWR012" H 6200 1800 50  0001 C CNN
 F 1 "GND" H 6200 1900 50  0000 C CNN
 F 2 "" H 6200 2050 50  0000 C CNN
@@
 $EndComp
 $Comp
+L VCC #PWR013
+U 1 1 580E7B51
+P 2100 1350
+F 0 "#PWR013" H 2100 1200 50  0001 C CNN
+F 1 "VCC" H 2100 1500 50  0000 C CNN
+F 2 "" H 2100 1350 50  0000 C CNN
+F 3 "" H 2100 1350 50  0000 C CNN
+	1    2100 1350
+	1    0    0    -1
+$EndComp
+$Comp
 L VCC #PWR014
-U 1 1 580E8E28
-P 6200 3550
-F 0 "#PWR014" H 6200 3400 50  0001 C CNN
-F 1 "VCC" H 6200 3700 50  0000 C CNN
-F 2 "" H 6200 3550 50  0000 C CNN
-F 3 "" H 6200 3550 50  0000 C CNN
-	1    6200 3550
+U 1 1 580E9B1D
+P 4500 1300
+F 0 "#PWR014" H 4500 1150 50  0001 C CNN
+F 1 "VCC" H 4500 1450 50  0000 C CNN
+F 2 "" H 4500 1300 50  0000 C CNN
+F 3 "" H 4500 1300 50  0000 C CNN
+	1    4500 1300
+	1    0    0    -1
+$EndComp
+$Comp
+L GND #PWR015
+U 1 1 580E9B87
+P 4500 2600
+F 0 "#PWR015" H 4500 2350 50  0001 C CNN
+F 1 "GND" H 4500 2450 50  0000 C CNN
+F 2 "" H 4500 2600 50  0000 C CNN
+F 3 "" H 4500 2600 50  0000 C CNN
+	1    4500 2600
+	1    0    0    -1
+$EndComp
+$Comp
+L VCC #PWR016
+U 1 1 580E9C6A
+P 4500 3150
+F 0 "#PWR016" H 4500 3000 50  0001 C CNN
+F 1 "VCC" H 4500 3300 50  0000 C CNN
+F 2 "" H 4500 3150 50  0000 C CNN
+F 3 "" H 4500 3150 50  0000 C CNN
+	1    4500 3150
+	1    0    0    -1
+$EndComp
+$Comp
+L GND #PWR017
+U 1 1 580E9C8D
+P 4500 4450
+F 0 "#PWR017" H 4500 4200 50  0001 C CNN
+F 1 "GND" H 4500 4300 50  0000 C CNN
+F 2 "" H 4500 4450 50  0000 C CNN
+F 3 "" H 4500 4450 50  0000 C CNN
+	1    4500 4450
+	1    0    0    -1
+$EndComp
+NoConn ~ 2100 1450
+NoConn ~ 2100 1550
+NoConn ~ 2100 1750
+NoConn ~ 2100 1850
+$Comp
+L GND #PWR018
+U 1 1 5901CAA6
+P 1250 2600
+F 0 "#PWR018" H 1250 2350 50  0001 C CNN
+F 1 "GND" H 1250 2450 50  0000 C CNN
+F 2 "" H 1250 2600 50  0000 C CNN
+F 3 "" H 1250 2600 50  0000 C CNN
+	1    1250 2600
+	-1   0    0    1
+$EndComp
+Text Label 1250 2700 2    60   ~ 0
+~EN
+Text Label 1250 2800 2    60   ~ 0
+B2
+Text Label 1250 2900 2    60   ~ 0
+B1
+Text Label 1250 3000 2    60   ~ 0
+A2
+Text Label 1250 3100 2    60   ~ 0
+A1
+$Comp
+L CONN_01X06 P4
+U 1 1 5901CA9B
+P 1450 2850
+F 0 "P4" H 1450 3200 50  0000 C CNN
+F 1 "KEYMAN64" V 1550 2850 50  0000 C CNN
+F 2 "Pin_Headers:Pin_Header_Angled_1x06_Pitch2.54mm" H 1450 2850 50  0001 C CNN
+F 3 "" H 1450 2850 50  0000 C CNN
+	1    1450 2850
+	1    0    0    -1
+$EndComp
+$Comp
+L GND #PWR019
+U 1 1 580E8E34
+P 6200 3750
+F 0 "#PWR019" H 6200 3500 50  0001 C CNN
+F 1 "GND" H 6200 3600 50  0000 C CNN
+F 2 "" H 6200 3750 50  0000 C CNN
+F 3 "" H 6200 3750 50  0000 C CNN
+	1    6200 3750
 	1    0    0    -1
 $EndComp
@@
 F 0 "C2" H 6210 3720 50  0000 L CNN
 F 1 "100n" H 6210 3570 50  0000 L CNN
-F 2 "Capacitors_ThroughHole:C_Disc_D3_P2.5" H 6200 3650 50  0001 C CNN
+F 2 "Capacitors_ThroughHole:C_Disc_D3.0mm_W1.6mm_P2.50mm" H 6200 3650 50  0001 C CNN
 F 3 "" H 6200 3650 50  0000 C CNN
 	1    6200 3650
@@
 $EndComp
 $Comp
-L GND #PWR015
-U 1 1 580E8E34
-P 6200 3750
-F 0 "#PWR015" H 6200 3500 50  0001 C CNN
-F 1 "GND" H 6200 3600 50  0000 C CNN
-F 2 "" H 6200 3750 50  0000 C CNN
-F 3 "" H 6200 3750 50  0000 C CNN
-	1    6200 3750
-	1    0    0    -1
-$EndComp
-$Comp
-L VCC #PWR016
-U 1 1 580E7B51
-P 2100 1350
-F 0 "#PWR016" H 2100 1200 50  0001 C CNN
-F 1 "VCC" H 2100 1500 50  0000 C CNN
-F 2 "" H 2100 1350 50  0000 C CNN
-F 3 "" H 2100 1350 50  0000 C CNN
-	1    2100 1350
-	1    0    0    -1
-$EndComp
-$Comp
-L VCC #PWR017
-U 1 1 580E9B1D
-P 4500 1300
-F 0 "#PWR017" H 4500 1150 50  0001 C CNN
-F 1 "VCC" H 4500 1450 50  0000 C CNN
-F 2 "" H 4500 1300 50  0000 C CNN
-F 3 "" H 4500 1300 50  0000 C CNN
-	1    4500 1300
-	1    0    0    -1
-$EndComp
-$Comp
-L GND #PWR018
-U 1 1 580E9B87
-P 4500 2600
-F 0 "#PWR018" H 4500 2350 50  0001 C CNN
-F 1 "GND" H 4500 2450 50  0000 C CNN
-F 2 "" H 4500 2600 50  0000 C CNN
-F 3 "" H 4500 2600 50  0000 C CNN
-	1    4500 2600
-	1    0    0    -1
-$EndComp
-$Comp
-L VCC #PWR019
-U 1 1 580E9C6A
-P 4500 3150
-F 0 "#PWR019" H 4500 3000 50  0001 C CNN
-F 1 "VCC" H 4500 3300 50  0000 C CNN
-F 2 "" H 4500 3150 50  0000 C CNN
-F 3 "" H 4500 3150 50  0000 C CNN
-	1    4500 3150
-	1    0    0    -1
-$EndComp
-$Comp
-L GND #PWR020
-U 1 1 580E9C8D
-P 4500 4450
-F 0 "#PWR020" H 4500 4200 50  0001 C CNN
-F 1 "GND" H 4500 4300 50  0000 C CNN
-F 2 "" H 4500 4450 50  0000 C CNN
-F 3 "" H 4500 4450 50  0000 C CNN
-	1    4500 4450
-	1    0    0    -1
-$EndComp
-NoConn ~ 2100 1450
-NoConn ~ 2100 1550
-NoConn ~ 2100 1750
-NoConn ~ 2100 1850
+L VCC #PWR020
+U 1 1 580E8E28
+P 6200 3550
+F 0 "#PWR020" H 6200 3400 50  0001 C CNN
+F 1 "VCC" H 6200 3700 50  0000 C CNN
+F 2 "" H 6200 3550 50  0000 C CNN
+F 3 "" H 6200 3550 50  0000 C CNN
+	1    6200 3550
+	1    0    0    -1
+$EndComp
 $EndSCHEMATC
